File: pcb_design/sema/SemaV1.kicad_pcb (KiCad board)
At the start: 2 copper layers, 74.9 x 72.4 mm, 26 parts, among them IC1 PIC24FJ64GA002-I_SP, J1 Conn_01x05_Pin, J15 Conn_01x01_Pin, J16 Conn_01x01_Pin, J19 Conn_01x02_Pin, J20 Conn_01x02_Pin, U1 ESP8266-01_ESP-01

Commit message: Dodavanje pcb fajla sa rutiranim komponentama
Sitne izmjene sa semi
Parts:
- removed U2: ~, Edge_Connector_Library:Edge_Connector
- added U1: ~, Edge_Connector_Library:Edge_Connector, F.Cu at (104.8, 128.3)
- C1, C2, C4, C5: footprint CAP_0.1u:CAPC5750X270N -> CAP_0.1uF:C1812
- C3: footprint CAP_10u:C2220_FT -> CAP_10uF:C1812
- J1: value Conn_01x05_Pin -> PICkit3 - ICSP
- moved R3 33.0 mm to (124.6, 85.1), turned to 180 degrees
- moved TP_RXD_WiFi1 31.9 mm to (144.8, 101.6)
- moved RST1 29.9 mm to (108.0, 97.8), turned to 0 degrees
- moved R1 26.5 mm to (134.6, 63.5)
- moved R4 21.6 mm to (124.5, 90.2)
- moved J19 17.1 mm to (125.7, 59.7), turned to 180 degrees
- moved WiFi1 15.7 mm to (99.6, 87.6)
- moved C4 15.1 mm to (125.0, 68.6)
- moved C5 14.3 mm to (108.4, 77.5), turned to 180 degrees
- moved I2C1 13.5 mm to (157.5, 88.9)
- moved TP_SCL1 12.8 mm to (147.3, 106.7)
- moved TP_TXD_WiFI1 12.7 mm to (123.2, 101.6)
- moved SPI1 12.1 mm to (157.5, 69.8)
- moved UART1 12.1 mm to (157.5, 80.0)
- moved R5 11.9 mm to (139.2, 105.4), turned to 180 degrees
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- renumbered J20 to RST1, J16 to TP_RXD_WiFi1, TP_1 to TP_SCL1, TP_2 to TP_SDA1, J15 to TP_TXD_WiFI1, U1 to WiFi1
Connections:
- net /SCL_2 renamed /SCL_1
- net /SDA_2 renamed /SDA_1
Routing:
- net Net-(IC1-AN4/C1IN-/RP2/SDA2/CN6/RB2): track 123.8 -> 73.0 mm, vias 1 -> 2
- net Net-(RST1-Pin_2): track 53.2 -> 24.6 mm
- net Net-(IC1-PGC3/EMUC3/RP6/ASCL1/CN24/PMD6/RB6): track 37.2 -> 60.2 mm
- net Net-(IC1-AN5/C1IN+/RP3/SCL2/CN7/RB3): track 78.1 -> 57.5 mm, vias 1 -> 2
- net Net-(IC1-RP7/INT0/CN23/PMD5/RB7): track 40.0 -> 56.4 mm
- net VDD: track 197.1 -> 187.7 mm, vias 0 -> 3
- net /RX: track 30.2 -> 20.8 mm
- net /SDA_1: track 31.3 -> 22.4 mm
- net /TX: track 29.1 -> 20.8 mm
- net GND: track 175.3 -> 183.0 mm, vias 4 -> 3
- net /SCL_1: track 32.8 -> 25.4 mm, vias 0 -> 2
- net Net-(IC1-VSS_2): track 10.7 -> 3.73 mm
- net Net-(WiFi1-EN): track 18.6 -> 12.1 mm
- net /SCK: track 29.1 -> 22.9 mm
- net /SS: track 29.1 -> 22.9 mm
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- added copper zone on B.Cu, net GND
- added copper zone on F.Cu, net GND
Other:
- board size 74.9 x 72.4 mm -> 62.4 x 72.6 mm
- board text added: "2024."
- board text added: "ETF BL"
- board text added: "MCLR VDD VSS PGD PCG"
- board text added: "Nemanja T. Bozana S. Dajana L."
- board text added: "SDA SCL"
- board text added: "SDI SDO SCK SS"
- board text added: "TX RX"
