File: pcb_design/kicad_schematic_pcb/control_board.kicad_sch (KiCad schematic)
At the start: 26 parts, among them IC1 PIC24FJ64GA002-I_SP, J1 PICkit3 - ICSP, J19 Conn_01x02_Pin

Commit message: Issue #22 : Rutiranje PCB-a
 - Izmjene footprint-a svih otpornika

 - Izmjene rutiranja komponenata u skladu sa primjedbama
Parts:
- R1, R3, R4: footprint RES_10k:RESC6432X120N -> RES_10k_new:RESC2012X65N
- R2: footprint RES_470:RESC6332X65N -> RES_470_new:ERA6VK
- R5, R6, R7, R8: footprint RES_4k7:RESC6432X65N -> RES_4k7_new:ERA6AEB1020V
Changed lines of the file:
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@@
       (effects (font (size 1.27 1.27)) (justify left))
     )
-    (property "Footprint" "RES_10k:RESC6432X120N" (at 215.392 100.33 90)
+    (property "Footprint" "RES_10k_new:RESC2012X65N" (at 215.392 100.33 90)
       (effects (font (size 1.27 1.27)) hide)
     )
@@
       (effects (font (size 1.27 1.27)) (justify left))
     )
-    (property "Footprint" "RES_10k:RESC6432X120N" (at 54.102 39.37 90)
+    (property "Footprint" "RES_10k_new:RESC2012X65N" (at 54.102 39.37 90)
       (effects (font (size 1.27 1.27)) hide)
     )
@@
       (effects (font (size 1.27 1.27)) (justify left))
     )
-    (property "Footprint" "RES_4k7:RESC6432X65N" (at 238.252 67.31 90)
+    (property "Footprint" "RES_4k7_new:ERA6AEB1020V" (at 238.252 67.31 90)
       (effects (font (size 1.27 1.27)) hide)
     )
@@
       (effects (font (size 1.27 1.27)) (justify left))
     )
-    (property "Footprint" "RES_4k7:RESC6432X65N" (at 87.122 107.95 90)
+    (property "Footprint" "RES_4k7_new:ERA6AEB1020V" (at 87.122 107.95 90)
       (effects (font (size 1.27 1.27)) hide)
     )
@@
       (effects (font (size 1.27 1.27)) (justify left))
     )
-    (property "Footprint" "RES_10k:RESC6432X120N" (at 220.472 97.79 90)
+    (property "Footprint" "RES_10k_new:RESC2012X65N" (at 220.472 97.79 90)
       (effects (font (size 1.27 1.27)) hide)
     )
@@
       (effects (font (size 1.27 1.27)) (justify left))
     )
-    (property "Footprint" "RES_4k7:RESC6432X65N" (at 230.632 68.58 90)
+    (property "Footprint" "RES_4k7_new:ERA6AEB1020V" (at 230.632 68.58 90)
       (effects (font (size 1.27 1.27)) hide)
     )
@@
       (effects (font (size 1.27 1.27)))
     )
-    (property "Footprint" "RES_470:RESC6332X65N" (at 85.09 51.308 90)
+    (property "Footprint" "RES_470_new:ERA6VK" (at 85.09 51.308 90)
       (effects (font (size 1.27 1.27)) hide)
     )
@@
       (effects (font (size 1.27 1.27)) (justify left))
     )
-    (property "Footprint" "RES_4k7:RESC6432X65N" (at 79.502 111.76 90)
-      (effects (font (size 1.27 1.27)) hide)
-    )
+    (property "Footprint" "RES_4k7_new:ERA6AEB1020V" (at 79.502 111.76 90)
+      (effects (font (size 1.27 1.27)) hide)
+    )
